Commit message: ur5 urdf add pole

File: mujoco_models/urdfs/ur5_joint_limited_robot.urdf.xacro (robot description, xacro)
@@ -20,6 +20,28 @@
   <joint name="world_joint" type="fixed">
     <parent link="world" />
+    <child link = "base_pole" />
+    <origin xyz="0.0 0.0 0.45" rpy="0.0 0.0 0.0" />
+  </joint>
+  <link name="base_pole">
+    <visual>
+      <origin xyz="0 0 0.0" rpy="0 0 0" />
+      <geometry>
+        <cylinder radius="0.08" length="0.9" />
+      </geometry>
+      <material name="grey">
+        <color rgba="0.4 0.4 0.4 1.0"/>
+      </material>
+    </visual>
+    <collision>
+      <origin xyz="0 0 0.0" rpy="0 0 0"/>
+      <geometry>
+        <cylinder radius="0.08" length="0.9"/>
+      </geometry>
+    </collision>
+  </link>
+  <joint name="base_pole_joint" type="fixed">
+    <parent link="base_pole" />
     <child link = "base_link" />
-    <origin xyz="0.0 0.0 0.0" rpy="0.0 0.0 0.0" />
+    <origin xyz="0.0 0.0 0.45" rpy="0.0 0.0 0.0" />
   </joint>
 </robot>
