Commit message: update panda_arm urdf

File: ros_models/urdfs/panda.urdf.xacro (robot description, xacro)
@@ -10,13 +10,13 @@
   <!-- base -->
   <link name="world" />
+  <link name="robot0_base_link" />
   <joint name="robot0_base_joint" type="fixed">
     <origin xyz="-0.56 0.0 0.913" rpy="0 0 0"/>
-    <!-- <origin xyz="0.0 0.0 0.913" rpy="0 0 0"/> -->
     <parent link="world"/>
-    <child link="robot0_link0"/>
+    <child link="robot0_base_link"/>
   </joint>
-  <xacro:base_platform prefix="robot0_" attach_link="robot0_link0" />
+  <xacro:base_platform prefix="robot0_" attach_link="robot0_base_link" />
   <!-- arm -->
-  <xacro:panda_arm arm_id="robot0" connected_to="world" xyz="-0.56 0.0 0.913" rpy="0 0 0"/>
+  <xacro:panda_arm arm_id="robot0" connected_to="robot0_base_link" />
   <!-- gripper -->
   <link name="robot0_right_hand" /><!-- could add camera with this link -->
@@ -26,8 +26,9 @@
     <origin xyz="0 0 0.1065" rpy="0 0 -0.7858908" />
   </joint>
-  <xacro:hand ns="gripper0" rpy="0 0 ${-pi / 4}" connected_to="robot0_right_hand"/>
+  <!-- <xacro:hand ns="gripper0" rpy="0 0 ${-pi / 2}" connected_to="robot0_right_hand" safety_distance="0.03"/> -->
+  <xacro:hand ns="gripper0" rpy="0 0 ${-pi / 4}" connected_to="robot0_link8" safety_distance="0.03"/>
   <link name="gripper0_right_gripper" /><!-- rename grippe0_hand link -->
   <joint name="gripper0_right_gripper_joint" type="fixed">
-    <parent link="gripper0_hand" />
+    <parent link="robot0_right_hand" />
     <child link="gripper0_right_gripper" />
     <origin xyz="0 0 0" rpy="0 0 0" />

File: ros_models/urdfs/panda/hand.xacro (robot description, xacro)
@@ -1,5 +1,6 @@
 <?xml version="1.0" encoding="utf-8"?>
 <robot xmlns:xacro="http://www.ros.org/wiki/xacro" name="hand">
-  <xacro:macro name="hand" params="connected_to:='' ns:='' rpy:='0 0 0' xyz:='0 0 0' ">
+  <!-- safety_distance: Minimum safety distance in [m] by which the collision volumes are expanded and which is enforced during robot motions -->
+  <xacro:macro name="hand" params="connected_to:='' ns:='' rpy:='0 0 0' xyz:='0 0 0' safety_distance:=0">
     <xacro:unless value="${connected_to == ''}">
       <joint name="${ns}_hand_joint" type="fixed">
@@ -12,34 +13,55 @@
       <visual>
         <geometry>
-          <mesh filename="package://franka_panda_description/meshes/visual/hand.dae"/>
+          <mesh filename="package://franka_description/meshes/visual/hand.dae"/>
+        </geometry>
+      </visual>
+      <collision>
+        <origin xyz="0 0 0.04" rpy="0 ${pi/2} ${pi/2}"/>
+        <geometry>
+          <cylinder radius="${0.04+safety_distance}" length="0.1" />
+        </geometry>
+      </collision>
+      <collision>
+        <origin xyz="0 -0.05 0.04" rpy="0 0 0"/>
+        <geometry>
+          <sphere radius="${0.04+safety_distance}"  />
+        </geometry>
+      </collision>
+      <collision>
+        <origin xyz="0 0.05 0.04" rpy="0 0 0"/>
+        <geometry>
+          <sphere radius="${0.04+safety_distance}"  />
+        </geometry>
+      </collision>
+      <collision>
+        <origin xyz="0 0 0.1" rpy="0 ${pi/2} ${pi/2}"/>
+        <geometry>
+          <cylinder radius="${0.02+safety_distance}" length="0.1" />
+        </geometry>
+      </collision>
+      <collision>
+        <origin xyz="0 -0.05 0.1" rpy="0 0 0"/>
+        <geometry>
+          <sphere radius="${0.02+safety_distance}"  />
+        </geometry>
+      </collision>
+      <collision>
+        <origin xyz="0 0.05 0.1" rpy="0 0 0"/>
+        <geometry>
+          <sphere radius="${0.02+safety_distance}"  />
+        </geometry>
+      </collision>
+    </link>
+    <link name="${ns}_leftfinger">
+      <visual>
+        <geometry>
+          <mesh filename="package://franka_description/meshes/visual/finger.dae"/>
         </geometry>
       </visual>
       <collision>
         <geometry>
-          <mesh filename="package://franka_panda_description/meshes/collision/hand.stl"/>
+          <mesh filename="package://franka_description/meshes/visual/finger.dae"/>
         </geometry>
       </collision>
-      <inertial>
-        <origin xyz="0 0 0" rpy="0 0 0"/>
-        <mass value="0.68"/>
-        <inertia ixx="0.1" ixy="0.0" ixz="0.0" iyy="0.1" iyz="0.0" izz="0.1"/>
-      </inertial>
-    </link>
-    <link name="${ns}_leftfinger">
-      <visual>
-        <geometry>
-          <mesh filename="package://franka_panda_description/meshes/visual/finger.dae"/>
-        </geometry>
-      </visual>
-      <collision>
-        <geometry>
-          <mesh filename="package://franka_panda_description/meshes/collision/finger.stl"/>
-        </geometry>
-      </collision>
-      <inertial>
-        <origin xyz="0 0 0" rpy="0 0 0"/>
-        <mass value="0.01"/>
-        <inertia ixx="0.1" ixy="0.0" ixz="0.0" iyy="0.1" iyz="0.0" izz="0.1"/>
-      </inertial>
     </link>
     <link name="${ns}_rightfinger">
@@ -47,5 +69,5 @@
         <origin xyz="0 0 0" rpy="0 0 ${pi}"/>
         <geometry>
-          <mesh filename="package://franka_panda_description/meshes/visual/finger.dae"/>
+          <mesh filename="package://franka_description/meshes/visual/finger.dae"/>
         </geometry>
       </visual>
@@ -53,13 +75,8 @@
         <origin xyz="0 0 0" rpy="0 0 ${pi}"/>
         <geometry>
-          <mesh filename="package://franka_panda_description/meshes/collision/finger.stl"/>
+          <mesh filename="package://franka_description/meshes/visual/finger.dae"/>
         </geometry>
       </collision>
-      <inertial>
-        <origin xyz="0 0 0" rpy="0 0 0"/>
-        <mass value="0.01"/>
-        <inertia ixx="0.1" ixy="0.0" ixz="0.0" iyy="0.1" iyz="0.0" izz="0.1"/>
-      </inertial>
-    </link>
+   </link>
     <joint name="${ns}_finger_joint1" type="prismatic">
       <parent link="${ns}_hand"/>
@@ -68,5 +85,4 @@
       <axis xyz="0 1 0"/>
       <limit effort="20" lower="0.0" upper="0.04" velocity="0.2"/>
-      <dynamics damping="500.0" friction="0.0"/>
     </joint>
     <joint name="${ns}_finger_joint2" type="prismatic">
@@ -76,5 +92,4 @@
       <axis xyz="0 -1 0"/>
       <limit effort="20" lower="0.0" upper="0.04" velocity="0.2"/>
-      <dynamics damping="500.0" friction="0.0"/>
       <mimic joint="${ns}_finger_joint1" />
     </joint>

File: ros_models/urdfs/panda/panda_arm.urdf.xacro (robot description, xacro)
@@ -1,11 +1,5 @@
-<?xml version='1.0' ?>
+<?xml version='1.0' encoding='utf-8'?>
 <robot xmlns:xacro="http://www.ros.org/wiki/xacro" name="panda">
-    <xacro:arg name="load_gazebo" default="false"/>
-    <xacro:include filename="$(find franka_panda_description)/robots/panda_arm.xacro"/>
-    <xacro:if value="$(arg load_gazebo)">
-        <xacro:panda_arm in_gazebo="true" />
-    </xacro:if>
-    <xacro:unless value="$(arg load_gazebo)">
-        <xacro:panda_arm />
-    </xacro:unless>
+  <xacro:include filename="$(find franka_description)/robots/panda_arm.xacro" />
+  <xacro:panda_arm safety_distance="0.03"/>
 </robot>

File: ros_models/urdfs/panda/panda_arm.xacro (robot description, xacro)
@@ -1,21 +1,14 @@
-<?xml version='1.0'?>
+<?xml version='1.0' encoding='utf-8'?>
 <robot xmlns:xacro="http://www.ros.org/wiki/xacro" name="panda">
-  <xacro:macro name="panda_arm" params="arm_id:='panda' description_pkg:='franka_panda_description' connected_to:=''  in_gazebo='false' xyz:='0 0 0' rpy:='0 0 0'">
-    <!-- If using custom frame with ${connected_to} param, make sure 'world' frame exists in its TF tree -->
-    <xacro:if value="${connected_to == ''}">
-      <link name="world" />
-      <xacro:property name="base_frame_name" value="world"/>
-    </xacro:if>
-    <xacro:unless value="${connected_to == ''}">
-      <xacro:property name="base_frame_name" value="${connected_to}"/>
+  <!-- safety_distance: Minimum safety distance in [m] by which the collision volumes are expanded and which is enforced during robot motions -->
+  <!-- arm_id: Namespace of the panda arm. Serves to differentiate between arms in case of multiple instances. -->
+  <xacro:macro name="panda_arm" params="arm_id:='panda' description_pkg:='franka_description' connected_to:='' xyz:='0 0 0' rpy:='0 0 0' safety_distance:=0">
+    <xacro:unless value="${not connected_to}">
+      <joint name="${arm_id}_joint_${connected_to}" type="fixed">
+        <parent link="${connected_to}"/>
+        <child link="${arm_id}_link0"/>
+        <origin rpy="${rpy}" xyz="${xyz}"/>
+      </joint>
     </xacro:unless>
-    <joint name="${arm_id}_to_${base_frame_name}" type="fixed">
-      <parent link="${base_frame_name}"/>
-      <child link="${arm_id}_link0"/>
-      <origin rpy="${rpy}" xyz="${xyz}"/>
-      <xacro:unless value="${in_gazebo == 'false'}">
-        <dynamics damping="1.0"/>
-      </xacro:unless>
-    </joint>
     <link name="${arm_id}_link0">
       <visual>
@@ -25,15 +18,21 @@
       </visual>
       <collision>
-        <geometry>
-          <mesh filename="package://${description_pkg}/meshes/collision/link0.stl"/>
-        </geometry>
-      </collision>
-      <xacro:unless value="${in_gazebo == 'false'}">
-        <inertial>
-          <origin xyz="0 0 0" rpy="0 0 0"/>
-          <mass value="3.06"/>
-          <inertia ixx="0.3" ixy="0.0" ixz="0.0" iyy="0.3" iyz="0.0" izz="0.3"/>
-        </inertial>
-      </xacro:unless>
+        <origin xyz="-0.075 0 0.06" rpy="0 ${pi/2} 0"/>
+        <geometry>
+          <cylinder radius="${0.06+safety_distance}" length="0.03" />
+        </geometry>
+      </collision>
+      <collision>
+        <origin xyz="-0.06 0 0.06" rpy="0 0 0"/>
+        <geometry>
+          <sphere radius="${0.06+safety_distance}" />
+        </geometry>
+      </collision>
+      <collision>
+        <origin xyz="-0.09 0 0.06" rpy="0 0 0"/>
+        <geometry>
+          <sphere radius="${0.06+safety_distance}" />
+        </geometry>
+      </collision>
     </link>
     <link name="${arm_id}_link1">
@@ -44,13 +43,21 @@
       </visual>
       <collision>
-        <geometry>
-          <mesh filename="package://${description_pkg}/meshes/collision/link1.stl"/>
-        </geometry>
-      </collision>
-      <inertial>
-        <origin xyz="3.875e-03 2.081e-03 -0.1750" rpy="0 0 0"/>
-        <mass value="4.970684"/>
-        <inertia ixx="7.0337e-01" ixy="-1.3900e-04" ixz="6.7720e-03" iyy="7.0661e-01" iyz="1.9169e-02" izz="9.1170e-03"/>
-      </inertial>
+        <origin xyz="0 0 -0.1915" rpy="0 0 0"/>
+        <geometry>
+          <cylinder radius="${0.06+safety_distance}" length="0.2830" />
+        </geometry>
+      </collision>
+      <collision>
+        <origin xyz="0 0 -0.333" rpy="0 0 0"/>
+        <geometry>
+          <sphere radius="${0.06+safety_distance}" />
+        </geometry>
+      </collision>
+      <collision>
+        <origin xyz="0 0 -0.05" rpy="0 0 0"/>
+        <geometry>
+          <sphere radius="${0.06+safety_distance}" />
+        </geometry>
+      </collision>
     </link>
     <joint name="${arm_id}_joint1" type="revolute">
@@ -61,5 +68,4 @@
       <axis xyz="0 0 1"/>
       <limit effort="87" lower="-2.8973" upper="2.8973" velocity="2.1750"/>
-      <dynamics damping="10.0" friction="5.0"/>
     </joint>
     <link name="${arm_id}_link2">
@@ -70,13 +76,21 @@
       </visual>
       <collision>
-        <geometry>
-          <mesh filename="package://${description_pkg}/meshes/collision/link2.stl"/>
-        </geometry>
-      </collision>
-      <inertial>
-        <origin xyz="-3.141e-03 -2.872e-02 3.495e-03" rpy="0 0 0"/>
-        <mass value="0.646926"/>
-        <inertia ixx="7.9620e-03" ixy="-3.9250e-03" ixz="1.0254e-02" iyy="2.8110e-02" iyz="7.0400e-04" izz="2.5995e-02"/>
-      </inertial>
+        <origin xyz="0 0 0" rpy="0 0 0"/>
+        <geometry>
+          <cylinder radius="${0.06+safety_distance}" length="0.12" />
+        </geometry>
+      </collision>
+      <collision>
+        <origin xyz="0 0 -0.06" rpy="0 0 0"/>
+        <geometry>
+          <sphere radius="${0.06+safety_distance}" />
+        </geometry>
+      </collision>
+      <collision>
+        <origin xyz="0 0 0.06" rpy="0 0 0"/>
+        <geometry>
+          <sphere radius="${0.06+safety_distance}" />
+        </geometry>
+      </collision>
     </link>
     <joint name="${arm_id}_joint2" type="revolute">
@@ -87,5 +101,4 @@
       <axis xyz="0 0 1"/>
       <limit effort="87" lower="-1.7628" upper="1.7628" velocity="2.1750"/>
-      <dynamics damping="5.0" friction="2.0"/>
     </joint>
     <link name="${arm_id}_link3">
@@ -96,13 +109,21 @@
       </visual>
       <collision>
-        <geometry>
-          <mesh filename="package://${description_pkg}/meshes/collision/link3.stl"/>
-        </geometry>
-      </collision>
-      <inertial>
-        <origin xyz="2.7518e-02 3.9252e-02 -6.6502e-02" rpy="0 0 0"/>
-        <mass value="3.228604"/>
-        <inertia ixx="3.7242e-02" ixy="-4.7610e-03" ixz="-1.1396e-02" iyy="3.6155e-02" iyz="-1.2805e-02" izz="1.0830e-02"/>
-      </inertial>
+        <origin xyz="0 0 -0.145" rpy="0 0 0"/>
+        <geometry>
+          <cylinder radius="${0.06+safety_distance}" length="0.15" />
+        </geometry>
+      </collision>
+      <collision>
+        <origin xyz="0 0 -0.22" rpy="0 0 0"/>
+        <geometry>
+          <sphere radius="${0.06+safety_distance}" />
+        </geometry>
+      </collision>
+      <collision>
+        <origin xyz="0 0 -0.07" rpy="0 0 0"/>
+        <geometry>
+          <sphere radius="${0.06+safety_distance}" />
+        </geometry>
+      </collision>
     </link>
     <joint name="${arm_id}_joint3" type="revolute">
@@ -113,5 +134,4 @@
       <axis xyz="0 0 1"/>
       <limit effort="87" lower="-2.8973" upper="2.8973" velocity="2.1750"/>
-      <dynamics damping="5.0" friction="2.0"/>
     </joint>
     <link name="${arm_id}_link4">
@@ -122,13 +142,21 @@
       </visual>
       <collision>
-        <geometry>
-          <mesh filename="package://${description_pkg}/meshes/collision/link4.stl"/>
-        </geometry>
-      </collision>
-      <inertial>
-        <origin xyz="-5.317e-02 1.04419e-01 2.7454e-02" rpy="0 0 0"/>
-        <mass value="3.587895"/>
-        <inertia ixx="2.5853e-02" ixy="7.7960e-03" ixz="-1.3320e-03" iyy="1.9552e-02" iyz="8.6410e-03" izz="2.8323e-02"/>
-      </inertial>
+        <origin xyz="0 0 0" rpy="0 0 0"/>
+        <geometry>
+          <cylinder radius="${0.06+safety_distance}" length="0.12" />
+        </geometry>
+      </collision>
+      <collision>
+        <origin xyz="0 0 0.06" rpy="0 0 0"/>
+        <geometry>
+          <sphere radius="${0.06+safety_distance}" />
+        </geometry>
+      </collision>
+      <collision>
+        <origin xyz="0 0 -0.06" rpy="0 0 0"/>
+        <geometry>
+          <sphere radius="${0.06+safety_distance}" />
+        </geometry>
+      </collision>
     </link>
     <joint name="${arm_id}_joint4" type="revolute">
@@ -139,5 +167,4 @@
       <axis xyz="0 0 1"/>
       <limit effort="87" lower="-3.0718" upper="-0.0698" velocity="2.1750"/>
-      <dynamics damping="1.0" friction="0.5"/>
     </joint>
     <link name="${arm_id}_link5">
@@ -148,13 +175,39 @@
       </visual>
       <collision>
-        <geometry>
-          <mesh filename="package://${description_pkg}/meshes/collision/link5.stl"/>
-        </geometry>
-      </collision>
-      <inertial>
-        <origin xyz="-1.1953e-02 4.1065e-02 -3.8437e-02" rpy="0 0 0"/>
-        <mass value="1.225946"/>
-        <inertia ixx="3.5549e-02" ixy="-2.1170e-03" ixz="-4.0370e-03" iyy="2.9474e-02" iyz="2.2900e-04" izz="8.6270e-03"/>
-      </inertial>
+        <origin xyz="0 0 -0.26" rpy="0 0 0"/>
+        <geometry>
+          <cylinder radius="${0.06+safety_distance}" length="0.1" />
+        </geometry>
+      </collision>
+      <collision>
+        <origin xyz="0 0 -0.31" rpy="0 0 0"/>
+        <geometry>
+          <sphere radius="${0.06+safety_distance}" />
+        </geometry>
+      </collision>
+      <collision>
+        <origin xyz="0 0 -0.21" rpy="0 0 0"/>
+        <geometry>
+          <sphere radius="${0.06+safety_distance}" />
+        </geometry>
+      </collision>
+      <collision>
+        <origin xyz="0 0.08 -0.13" rpy="0 0 0"/>
+        <geometry>
+          <cylinder radius="${0.025+safety_distance}" length="0.14" />
+        </geometry>
+      </collision>
+      <collision>
+        <origin xyz="0 0.08 -0.06" rpy="0 0 0"/>
+        <geometry>
+          <sphere radius="${0.025+safety_distance}" />
+        </geometry>
+      </collision>
+      <collision>
+        <origin xyz="0 0.08 -0.20" rpy="0 0 0"/>
+        <geometry>
+          <sphere radius="${0.025+safety_distance}" />
+        </geometry>
+      </collision>
     </link>
     <joint name="${arm_id}_joint5" type="revolute">
@@ -165,5 +218,4 @@
       <axis xyz="0 0 1"/>
       <limit effort="12" lower="-2.8973" upper="2.8973" velocity="2.6100"/>
-      <dynamics damping="2.0" friction="1.0"/>
     </joint>
     <link name="${arm_id}_link6">
@@ -174,13 +226,21 @@
       </visual>
       <collision>
-        <geometry>
-          <mesh filename="package://${description_pkg}/meshes/collision/link6.stl"/>
-        </geometry>
-      </collision>
-      <inertial>
-        <origin xyz="6.0149e-02 -1.4117e-02 -1.0517e-02" rpy="0 0 0"/>
-        <mass value="1.666555"/>
-        <inertia ixx="1.9640e-03" ixy="1.0900e-04" ixz="-1.1580e-03" iyy="4.3540e-03" iyz="3.4100e-04" izz="5.4330e-03"/>
-      </inertial>
+        <origin xyz="0 0 -0.03" rpy="0 0 0"/>
+        <geometry>
+          <cylinder radius="${0.05+safety_distance}" length="0.08" />
+        </geometry>
+      </collision>
+      <collision>
+        <origin xyz="0 0 0.01" rpy="0 0 0"/>
+        <geometry>
+          <sphere radius="${0.05+safety_distance}" />
+        </geometry>
+      </collision>
+      <collision>
+        <origin xyz="0 0 -0.07" rpy="0 0 0"/>
+        <geometry>
+          <sphere radius="${0.05+safety_distance}" />
+        </geometry>
+      </collision>
     </link>
     <joint name="${arm_id}_joint6" type="revolute">
@@ -191,5 +251,4 @@
       <axis xyz="0 0 1"/>
       <limit effort="12" lower="-0.0175" upper="3.7525" velocity="2.6100"/>
-      <dynamics damping="1.0" friction="0.5"/>
     </joint>
     <link name="${arm_id}_link7">
@@ -200,13 +259,21 @@
       </visual>
       <collision>
-        <geometry>
-          <mesh filename="package://${description_pkg}/meshes/collision/link7.stl"/>
-        </geometry>
-      </collision>
-      <inertial>
-        <origin xyz="1.0517e-02 -4.252e-03 6.1597e-02" rpy="0 0 0"/>
-        <mass value="7.35522e-01"/>
-        <inertia ixx="1.2516e-02" ixy="-4.2800e-04" ixz="-1.1960e-03" iyy="1.0027e-02" iyz="-7.4100e-04" izz="4.8150e-03"/>
-      </inertial>
+        <origin xyz="0 0 0.01" rpy="0 0 0"/>
+        <geometry>
+          <cylinder radius="${0.04+safety_distance}" length="0.14" />
+        </geometry>
+      </collision>
+      <collision>
+        <origin xyz="0 0 0.08" rpy="0 0 0"/>
+        <geometry>
+          <sphere radius="${0.04+safety_distance}"  />
+        </geometry>
+      </collision>
+      <collision>
+        <origin xyz="0 0 -0.06" rpy="0 0 0"/>
+        <geometry>
+          <sphere radius="${0.04+safety_distance}"  />
+        </geometry>
+      </collision>
     </link>
     <joint name="${arm_id}_joint7" type="revolute">
@@ -217,12 +284,24 @@
       <axis xyz="0 0 1"/>
       <limit effort="12" lower="-2.8973" upper="2.8973" velocity="2.6100"/>
-      <dynamics damping="1.0" friction="0.5"/>
     </joint>
     <link name="${arm_id}_link8">
-      <inertial>
-        <origin xyz="0 0 0" rpy="0 0 0"/>
-        <mass value="0.0"/>
-        <inertia ixx="0.001" ixy="0.0" ixz="0.0" iyy="0.001" iyz="0.0" izz="0.001"/>
-      </inertial>
+      <collision>
+        <origin xyz="0.0424 0.0424 -0.0250" rpy="${pi} ${pi/2} ${pi/2}"/>
+        <geometry>
+          <cylinder radius="${0.03+safety_distance}"  length="0.01" />
+        </geometry>
+      </collision>
+      <collision>
+        <origin xyz="0.0424 0.0424 -0.02" rpy="0 0 0"/>
+        <geometry>
+          <sphere radius="${0.03+safety_distance}"  />
+        </geometry>
+      </collision>
+      <collision>
+        <origin xyz="0.0424 0.0424 -0.03" rpy="0 0 0"/>
+        <geometry>
+          <sphere radius="${0.03+safety_distance}"  />
+        </geometry>
+      </collision>
     </link>
     <joint name="${arm_id}_joint8" type="fixed">
@@ -230,5 +309,4 @@
       <parent link="${arm_id}_link7"/>
       <child link="${arm_id}_link8"/>
-      <axis xyz="0 0 0"/>
     </joint>
   </xacro:macro>

File: ros_models/urdfs/panda/panda_arm_hand.urdf.xacro (robot description, xacro)
@@ -1,23 +1,7 @@
-<?xml version="1.0"?>
+<?xml version="1.0" encoding="utf-8"?>
 <robot xmlns:xacro="http://www.ros.org/wiki/xacro" name="panda">
-  <xacro:arg name="robot_name" default="panda"/>
-  <xacro:arg name="load_gripper" default="true"/>
-  <xacro:arg name="load_gazebo" default="false"/>
-  <xacro:arg name="use_gazebo_control" default="false"/>
-  <xacro:arg name="connected_to" default=""/> <!-- If using a different frame with ${connected_to} param, make sure 'world' frame exists in the TF tree -->
-  <xacro:include filename="$(find franka_panda_description)/robots/panda_arm.xacro"/>
-  <xacro:if value="$(arg load_gripper)">
-    <xacro:include filename="$(find franka_panda_description)/robots/hand.xacro"/>
-    <xacro:hand ns="panda" rpy="0 0 ${-pi/4}" connected_to="panda_link8"/>
-  </xacro:if>
-  <xacro:if value="$(arg load_gazebo)">
-    <xacro:include filename="$(find franka_panda_description)/robots/panda.gazebo.xacro"/>
-    <xacro:include filename="$(find franka_panda_description)/robots/panda.transmission.xacro"/>
-    <xacro:panda_arm in_gazebo="true"  connected_to="$(arg connected_to)"/>
-    <xacro:panda_gazebo robot_name="$(arg robot_name)" load_gripper="$(arg load_gripper)"/>
-    <xacro:panda_transmission robot_name="$(arg robot_name)" load_gripper="$(arg load_gripper)" use_gazebo_control="$(arg use_gazebo_control)"/>
-  </xacro:if>
-  <xacro:unless value="$(arg load_gazebo)">
-    <xacro:panda_arm />
-  </xacro:unless>
+  <xacro:include filename="$(find franka_description)/robots/panda_arm.xacro"/>
+  <xacro:include filename="$(find franka_description)/robots/hand.xacro"/>
+  <xacro:panda_arm safety_distance="0.03"/>
+  <xacro:hand ns="panda" rpy="0 0 ${-pi/4}" connected_to="panda_link8" safety_distance="0.03"/>
 </robot>
