Commit message: add jog and update initial joint positions

File: ros_models/urdfs/robotiq_2f_85/robotiq_arg2f_85_model_macro.xacro (robot description, xacro)
@@ -175,5 +175,5 @@
       <child link="${prefix}right_outer_knuckle" />
       <axis xyz="1 0 0" />
-      <limit lower="0" upper="0.80" velocity="2.0" effort="1000" />
+      <limit lower="0" upper="0.81" velocity="2.0" effort="1000" />
       <!-- (chongyi zheng): stand alone right_outer_knuckle_joint -->
       <!-- <mimic joint="${prefix}finger_joint" multiplier="1" offset="0" /> -->

File: ros_models/urdfs/robotiq_2f_85/robotiq_arg2f_transmission.xacro (robot description, xacro)
@@ -12,5 +12,5 @@
     </transmission>
     <!-- (chongyi zheng): add right_outer_knuckle_joint transimission -->
-    <transmission name="${prefix}right_outer_knuckle_joint">
+    <transmission name="${prefix}right_outer_knuckle_joint_trans">
       <type>transmission_interface/SimpleTransmission</type>
       <joint name="${prefix}right_outer_knuckle_joint">

Commit message: update mujoco and ros models

File: ros_models/urdfs/robotiq_2f_85/robotiq_arg2f_85_model_macro.xacro (robot description, xacro)
@@ -166,4 +166,5 @@
       <axis xyz="1 0 0" />
       <limit lower="0" upper="0.8" velocity="2.0" effort="1000" />
+      <!-- <limit lower="0" upper="0.73" velocity="2.0" effort="1000" /> -->
     </joint>
     <xacro:finger_joints prefix="${prefix}" fingerprefix="left" reflect="1.0" mimicjoint="${prefix}finger_joint"/>
@@ -176,4 +177,5 @@
       <axis xyz="1 0 0" />
       <limit lower="0" upper="0.81" velocity="2.0" effort="1000" />
+      <!-- <limit lower="0" upper="0.73" velocity="2.0" effort="1000" /> -->
       <!-- (chongyi zheng): stand alone right_outer_knuckle_joint -->
       <!-- <mimic joint="${prefix}finger_joint" multiplier="1" offset="0" /> -->
