Commit message: robotiq_3f urdf add transmissions

File: ros_models/urdfs/robotiq_3f/robotiq_hand_macro.urdf.xacro (robot description, xacro)
@@ -7,4 +7,5 @@
 -->
 <robot xmlns:xacro="http://www.ros.org/wiki/xacro" name="robotiq_hand">
+  <xacro:include filename="$(find bulldog_mujoco_ros)/ros_models/urdfs/robotiq_3f/robotiq-3f_gripper_transmission.xacro" />
   <xacro:macro name="robotiq_finger" params="prefix">
     <!-- Link list -->
@@ -522,4 +523,5 @@
       <!-- Limits: [0deg.,90deg.] -->
       <limit lower="0" upper="1.5708" effort="60" velocity="-1"/>
+      <mimic joint="${prefix}joint_1" multiplier="1" offset="0" />
     </joint>
     <gazebo reference="${prefix}joint_2">
@@ -535,4 +537,5 @@
       <!-- Limits: [-38deg.,60deg.] -->
       <limit lower="-0.6632" upper="1.0471" effort="60" velocity="-1"/>
+      <mimic joint="${prefix}joint_2" multiplier="-2" offset="0" />
     </joint>
     <gazebo reference="${prefix}joint_3">
@@ -698,4 +701,5 @@
       <!-- Limits: [-17deg.,17deg.] -->
       <limit lower="-0.2967" upper="0.2967" effort="60" velocity="-1"/>
+      <mimic joint="${prefix}joint_2" multiplier="-1" offset="0" />
     </joint>
     <gazebo reference="${prefix}palm_finger_2_joint">
@@ -715,4 +719,7 @@
     </gazebo>
     <!-- end of joint list -->
+    <!--Transmissions -->
+    <xacro:robotiq_transmission prefix="${prefix}"/>
+    <!-- end of transmission list -->
   </xacro:macro>
 </robot>
