Commit message: add ur5e_robotiq_3f_moveit_planning_and_execution.launch

File: ros_models/urdfs/robotiq_3f/robotiq-3f-gripper_articulated_macro.xacro (robot description, xacro)
@@ -6,6 +6,7 @@
 -->
 <robot xmlns:xacro="http://ros.org/wiki/xacro">
-        <xacro:include filename="$(find robotiq_3f_gripper_visualization)/cfg/robotiq-3f-gripper_finger_articulated_macro.xacro" />
-        <xacro:macro name="robotiq-3f-gripper_articulated" params="prefix">
+	<xacro:include filename="$(find robotiq_3f_gripper_visualization)/cfg/robotiq-3f-gripper_finger_articulated_macro.xacro" />
+  	<xacro:include filename="$(find bulldog_mujoco_ros)/ros_models/urdfs/robotiq_3f/robotiq-3f_gripper_transmission.xacro" />
+	<xacro:macro name="robotiq-3f-gripper_articulated" params="prefix">
         <xacro:robotiq-3f-gripper_finger_articulated prefix="${prefix}finger_1_"/>
         <xacro:robotiq-3f-gripper_finger_articulated prefix="${prefix}finger_2_"/>
@@ -15,5 +16,5 @@
 			<visual>
 				<geometry>
-                                        <mesh filename="package://robotiq_3f_gripper_visualization/meshes/robotiq-3f-gripper_articulated/visual/palm.dae" />
+                    <mesh filename="package://robotiq_3f_gripper_visualization/meshes/robotiq-3f-gripper_articulated/visual/palm.dae" />
 				</geometry>
 				<material name="gray">
@@ -23,5 +24,5 @@
 			<collision>
 				<geometry>
-                                        <mesh filename="package://robotiq_3f_gripper_visualization/meshes/robotiq-3f-gripper_articulated/collision/palm.STL" />
+                	<mesh filename="package://robotiq_3f_gripper_visualization/meshes/robotiq-3f-gripper_articulated/collision/palm.STL" />
 				</geometry>
 				<material name="yellow">
@@ -64,4 +65,7 @@
 		</joint>
 		<!-- end of joint list -->
+		<!-- transmissions -->
+    	<xacro:robotiq_transmission prefix="${prefix}"/>
+		<!-- end of transmissions -->
 	</xacro:macro>
 </robot>

File: ros_models/urdfs/robotiq_3f/robotiq-3f-gripper_finger_articulated_macro.xacro (robot description, xacro)
@@ -12,5 +12,5 @@
 				<origin xyz="0.020 0 0" rpy="0 0 0"/>
 				<geometry>
-                                        <mesh filename="package://robotiq_3f_gripper_visualization/meshes/robotiq-3f-gripper_articulated/visual/link_0.dae" />
+                    <mesh filename="package://robotiq_3f_gripper_visualization/meshes/robotiq-3f-gripper_articulated/visual/link_0.dae" />
 				</geometry>
 				<material name="gray">
@@ -21,5 +21,5 @@
 				<origin xyz="0.020 0 0" rpy="0 0 0"/>
 				<geometry>
-                                        <mesh filename="package://robotiq_3f_gripper_visualization/meshes/robotiq-3f-gripper_articulated/collision/link_0.STL" />
+                    <mesh filename="package://robotiq_3f_gripper_visualization/meshes/robotiq-3f-gripper_articulated/collision/link_0.STL" />
 				</geometry>
 				<material name="yellow">
@@ -37,5 +37,5 @@
 				<origin xyz="0.050 -.028 0" rpy="0 0 -0.52"/>
 				<geometry>
-                                        <mesh filename="package://robotiq_3f_gripper_visualization/meshes/robotiq-3f-gripper_articulated/visual/link_1.dae" />
+					<mesh filename="package://robotiq_3f_gripper_visualization/meshes/robotiq-3f-gripper_articulated/visual/link_1.dae" />
 				</geometry>
 				<material name="gray"/>
@@ -44,5 +44,5 @@
 				<origin xyz="0.050 -.028 0" rpy="0 0 -0.52"/>
 				<geometry>
-                                        <mesh filename="package://robotiq_3f_gripper_visualization/meshes/robotiq-3f-gripper_articulated/collision/link_1.STL" />
+					<mesh filename="package://robotiq_3f_gripper_visualization/meshes/robotiq-3f-gripper_articulated/collision/link_1.STL" />
 				</geometry>
 				<material name="yellow"/>
@@ -63,5 +63,5 @@
 				<origin xyz="0.039 0 0.0075" rpy="0 0 0"/>
 				<geometry>
-                                        <mesh filename="package://robotiq_3f_gripper_visualization/meshes/robotiq-3f-gripper_articulated/visual/link_2.dae" />
+					<mesh filename="package://robotiq_3f_gripper_visualization/meshes/robotiq-3f-gripper_articulated/visual/link_2.dae" />
 				</geometry>
 				<material name="gray"/>
@@ -70,5 +70,5 @@
 				<origin xyz="0.039 0 0.0075" rpy="0 0 0"/>
 				<geometry>
-                                        <mesh filename="package://robotiq_3f_gripper_visualization/meshes/robotiq-3f-gripper_articulated/collision/link_2.STL" />
+					<mesh filename="package://robotiq_3f_gripper_visualization/meshes/robotiq-3f-gripper_articulated/collision/link_2.STL" />
 				</geometry>
 				<material name="yellow"/>
@@ -84,5 +84,5 @@
 				<origin xyz="0 0 0" rpy="0 0 0.52"/>
 				<geometry>
-                                        <mesh filename="package://robotiq_3f_gripper_visualization/meshes/robotiq-3f-gripper_articulated/visual/link_3.dae" />
+					<mesh filename="package://robotiq_3f_gripper_visualization/meshes/robotiq-3f-gripper_articulated/visual/link_3.dae" />
 				</geometry>
 				<material name="gray"/>
@@ -91,5 +91,5 @@
 				<origin xyz="0 0 0" rpy="0 0 0.52"/>
 				<geometry>
-                                        <mesh filename="package://robotiq_3f_gripper_visualization/meshes/robotiq-3f-gripper_articulated/collision/link_3.STL" />
+					<mesh filename="package://robotiq_3f_gripper_visualization/meshes/robotiq-3f-gripper_articulated/collision/link_3.STL" />
 				</geometry>
 				<material name="yellow"/>

File: ros_models/urdfs/robotiq_3f/robotiq_hand_macro.urdf.xacro (robot description, xacro)
@@ -701,5 +701,5 @@
       <!-- Limits: [-17deg.,17deg.] -->
       <limit lower="-0.2967" upper="0.2967" effort="60" velocity="-1"/>
-      <mimic joint="${prefix}joint_2" multiplier="-1" offset="0" />
+      <mimic joint="${prefix}palm_finger_1_joint" multiplier="-1" offset="0" />
     </joint>
     <gazebo reference="${prefix}palm_finger_2_joint">

File: ros_models/urdfs/ur5e_robotiq_3f.urdf.xacro (robot description, xacro)
@@ -10,5 +10,5 @@
   <xacro:include filename="$(find bulldog_mujoco_ros)/ros_models/urdfs/ur5/ur5.urdf.xacro" />
   <!-- robotiq -->
-  <xacro:include filename="$(find bulldog_mujoco_ros)/ros_models/urdfs/robotiq_3f/robotiq_hand_macro.urdf.xacro" />
+  <xacro:include filename="$(find bulldog_mujoco_ros)/ros_models/urdfs/robotiq_3f/robotiq-3f-gripper_articulated_macro.xacro" />
   <!-- <body name="robot0_base" pos="-0.56 0.0 0.913">
       <inertial diaginertia="0 0 0" mass="0" pos="0 0 0" />
@@ -68,4 +68,5 @@
     <child link = "base_pole" />
     <origin xyz="0.0 0.0 0.45" rpy="0.0 0.0 0.0" />
+  <xacro:robotiq-3f-gripper_articulated prefix=""/>
   </joint>
   <link name="base_pole">
@@ -118,17 +119,18 @@
     <origin xyz="0 0.082 0" rpy="-1.5708 0 0" />
   </joint>
-  <xacro:robotiq_hand prefix="gripper0_" parent="robot0_right_hand" reflect="1">
+  <!-- <xacro:robotiq_hand prefix="gripper0_" parent="robot0_right_hand" reflect="1">
     <origin xyz="0 0 0.065" rpy="1.5708 0 2.3562" />
-  </xacro:robotiq_hand>
-  <!-- <joint name="gripper0_palm_joint" type="fixed">
+  </xacro:robotiq_hand> -->
+  <xacro:robotiq-3f-gripper_articulated prefix="gripper0_"/>
+  <joint name="gripper0_palm_joint" type="fixed">
     <parent link="robot0_right_hand" />
     <child link="gripper0_palm" />
     <origin xyz="0 0 0.065" rpy="1.5708 0 2.3562" />
-  </joint> -->
-  <link name="gripper0_tool0" />
+  </joint>
+  <!-- <link name="gripper0_tool0" />
   <joint name="gripper0_tool0_joint" type="fixed">
     <parent link="gripper0_palm" />
     <child link="gripper0_tool0" />
     <origin xyz="0 0.1 0" rpy="0 0 0" />
-  </joint>
+  </joint> -->
 </robot>
