Commit message: update ur5e_robotiq_3f

File: ros_models/urdfs/robotiq_3f/robotiq-3f-gripper_articulated_macro.xacro (robot description, xacro)
@@ -6,5 +6,5 @@
 -->
 <robot xmlns:xacro="http://ros.org/wiki/xacro">
-	<xacro:include filename="$(find robotiq_3f_gripper_visualization)/cfg/robotiq-3f-gripper_finger_articulated_macro.xacro" />
+	<xacro:include filename="$(find bulldog_mujoco_ros)/ros_models/urdfs/robotiq_3f/robotiq-3f-gripper_finger_articulated_macro.xacro" />
   	<xacro:include filename="$(find bulldog_mujoco_ros)/ros_models/urdfs/robotiq_3f/robotiq-3f_gripper_transmission.xacro" />
 	<xacro:macro name="robotiq-3f-gripper_articulated" params="prefix">
@@ -52,4 +52,5 @@
 			<origin xyz="-0.0455 0.0214 -0.036" rpy="0 3.1416 -1.57"/>
 			<limit lower="-0.192" upper="0.1784" effort="100" velocity="100"/>
+			<mimic joint="${prefix}palm_finger_1_joint" multiplier="-1" offset="0" />
 		</joint>
 		<joint name="${prefix}palm_finger_middle_joint" type="fixed">

File: ros_models/urdfs/robotiq_3f/robotiq-3f-gripper_finger_articulated_macro.xacro (robot description, xacro)
@@ -116,4 +116,5 @@
 			<origin xyz="0.050 -.028 0" rpy="0 0 -0.52"/>
 			<limit lower="0.0" upper="1.5708" effort="100" velocity="100"/>
+			<mimic joint="${prefix}joint_1" multiplier="1" offset="0" />
 		</joint>
 		<joint name="${prefix}joint_3" type="revolute">
@@ -123,4 +124,5 @@
 			<origin xyz="0.039 0 0" rpy="0 0 0"/>
 			<limit lower="-1.2217" upper="-0.0523" effort="100" velocity="100"/>
+			<mimic joint="${prefix}joint_2" multiplier="-2" offset="0" />
 		</joint>
 		<!-- end of joint list -->

File: ros_models/urdfs/robotiq_3f/robotiq_hand_macro.urdf.xacro (robot description, xacro)
@@ -36,8 +36,8 @@
       </inertial>
     </link>
-    <gazebo reference="${prefix}link_0">
-      <mu1>1.1</mu1>
-      <mu2>1.1</mu2>
-    </gazebo>
+    <!-- <gazebo reference="${prefix}link_0">
+      <mu1>1.1</mu1>
+      <mu2>1.1</mu2>
+    </gazebo> -->
     <!-- Link 1 -->
     <link name="${prefix}link_1">
@@ -69,8 +69,8 @@
       </inertial>
     </link>
-    <gazebo reference="${prefix}link_1">
-      <mu1>1.1</mu1>
-      <mu2>1.1</mu2>
-    </gazebo>
+    <!-- <gazebo reference="${prefix}link_1">
+      <mu1>1.1</mu1>
+      <mu2>1.1</mu2>
+    </gazebo> -->
     <!-- Link 2 -->
     <link name="${prefix}link_2">
@@ -100,8 +100,8 @@
       </inertial>
     </link>
-    <gazebo reference="${prefix}link_2">
-      <mu1>1.1</mu1>
-      <mu2>1.1</mu2>
-    </gazebo>
+    <!-- <gazebo reference="${prefix}link_2">
+      <mu1>1.1</mu1>
+      <mu2>1.1</mu2>
+    </gazebo> -->
     <!-- Link 3 -->
     <link name="${prefix}link_3">
@@ -131,10 +131,10 @@
       </inertial>
     </link>
-    <gazebo reference="${prefix}link_3">
-      <mu1>1.1</mu1>
-      <mu2>1.1</mu2>
-    </gazebo>
+    <!-- <gazebo reference="${prefix}link_3">
+      <mu1>1.1</mu1>
+      <mu2>1.1</mu2>
+    </gazebo> -->
     <!-- Link proximal actuating hinge -->
-    <link name="${prefix}link_proximal_actuating_hinge">
+    <!-- <link name="${prefix}link_proximal_actuating_hinge">
       <visual>
         <origin rpy="0 0 0" xyz="0.01429 0 0"/>
@@ -163,7 +163,7 @@
       <mu1>1.1</mu1>
       <mu2>1.1</mu2>
-    </gazebo>
+    </gazebo> -->
     <!-- Link paraproximal actuating hinge -->
-    <link name="${prefix}link_paraproximal_actuating_hinge">
+    <!-- <link name="${prefix}link_paraproximal_actuating_hinge">
       <visual>
         <origin rpy="0 0 0" xyz="0.01143 0 0"/>
@@ -180,5 +180,5 @@
       <inertial>
         <origin rpy="0 0 0" xyz="0.0064 0 0"/>
-        <!-- copied from proximal_actuating_hinge -->
+        copied from proximal_actuating_hinge
         <mass value="0.00362"/>
         <inertia ixx= "0.00000012043"
@@ -193,7 +193,7 @@
       <mu1>1.1</mu1>
       <mu2>1.1</mu2>
-    </gazebo>
+    </gazebo> -->
     <!-- Link proximal actuating bar -->
-    <link name="${prefix}link_proximal_actuating_bar">
+    <!-- <link name="${prefix}link_proximal_actuating_bar">
       <visual>
         <origin rpy="0 0 0" xyz="0.026789 0 0"/>
@@ -222,7 +222,7 @@
       <mu1>1.1</mu1>
       <mu2>1.1</mu2>
-    </gazebo>
+    </gazebo> -->
     <!-- Link paraproximal bar -->
-    <link name="${prefix}link_paraproximal_bar">
+    <!-- <link name="${prefix}link_paraproximal_bar">
       <visual>
         <origin rpy="0 0 0" xyz="0.02885 0 0"/>
@@ -251,7 +251,7 @@
       <mu1>1.1</mu1>
       <mu2>1.1</mu2>
-    </gazebo>
+    </gazebo> -->
     <!-- Link median actuating hinge -->
-    <link name="${prefix}link_median_actuating_hinge">
+    <!-- <link name="${prefix}link_median_actuating_hinge">
       <visual>
         <origin rpy="0 0 0" xyz="0 0 0"/>
@@ -280,7 +280,7 @@
       <mu1>1.1</mu1>
       <mu2>1.1</mu2>
-    </gazebo>
+    </gazebo> -->
     <!-- Link median bar -->
-    <link name="${prefix}link_median_bar">
+    <!-- <link name="${prefix}link_median_bar">
       <visual>
         <origin rpy="0 0 0" xyz="0.01905 0 0"/>
@@ -309,7 +309,7 @@
       <mu1>1.1</mu1>
       <mu2>1.1</mu2>
-    </gazebo>
+    </gazebo> -->
     <!-- Link paramedian hinge -->
-    <link name="${prefix}link_paramedian_hinge">
+    <!-- <link name="${prefix}link_paramedian_hinge">
       <visual>
         <origin rpy="0 0 0" xyz="0 0 0"/>
@@ -338,7 +338,7 @@
       <mu1>1.1</mu1>
       <mu2>1.1</mu2>
-    </gazebo>
+    </gazebo> -->
     <!-- Link median bar underactuated -->
-    <link name="${prefix}link_median_bar_underactuated">
+    <!-- <link name="${prefix}link_median_bar_underactuated">
       <visual>
         <origin rpy="0 0 0" xyz="0.01905 0 0"/>
@@ -367,7 +367,7 @@
       <mu1>1.1</mu1>
       <mu2>1.1</mu2>
-    </gazebo>
+    </gazebo> -->
     <!-- Link paradistal hinge -->
-    <link name="${prefix}link_paradistal_hinge">
+    <!-- <link name="${prefix}link_paradistal_hinge">
       <visual>
         <origin rpy="0 0 0" xyz="0 0 0"/>
@@ -396,9 +396,9 @@
       <mu1>1.1</mu1>
       <mu2>1.1</mu2>
-    </gazebo>
+    </gazebo> -->
     <!-- End of link list -->
     <!-- Joint list -->
     <!-- Joint proximal actuating hinge -->
-    <joint name="${prefix}joint_proximal_actuating_hinge" type="revolute">
+    <!-- <joint name="${prefix}joint_proximal_actuating_hinge" type="revolute">
       <parent link="${prefix}link_0"/>
       <child link="${prefix}link_proximal_actuating_hinge"/>
@@ -409,7 +409,7 @@
     <gazebo reference="${prefix}joint_proximal_actuating_hinge">
       <implicitSpringDamper>1</implicitSpringDamper>
-    </gazebo>
+    </gazebo> -->
     <!-- Joint paraproximal actuating hinge -->
-    <joint name="${prefix}joint_paraproximal_actuating_hinge" type="revolute">
+    <!-- <joint name="${prefix}joint_paraproximal_actuating_hinge" type="revolute">
       <parent link="${prefix}link_0"/>
       <child link="${prefix}link_paraproximal_actuating_hinge"/>
@@ -420,7 +420,7 @@
     <gazebo reference="${prefix}joint_paraproximal_actuating_hinge">
       <implicitSpringDamper>1</implicitSpringDamper>
-    </gazebo>
+    </gazebo> -->
     <!-- Joint proximal actuating bar -->
-    <joint name="${prefix}joint_proximal_actuating_bar" type="revolute">
+    <!-- <joint name="${prefix}joint_proximal_actuating_bar" type="revolute">
       <parent link="${prefix}link_proximal_actuating_hinge"/>
       <child link="${prefix}link_proximal_actuating_bar"/>
@@ -431,7 +431,7 @@
     <gazebo reference="${prefix}joint_proximal_actuating_bar">
       <implicitSpringDamper>1</implicitSpringDamper>
-    </gazebo>
+    </gazebo> -->
     <!-- Joint paraproximal bar -->
-    <joint name="${prefix}joint_paraproximal_bar" type="revolute">
+    <!-- <joint name="${prefix}joint_paraproximal_bar" type="revolute">
       <parent link="${prefix}link_paraproximal_actuating_hinge"/>
       <child link="${prefix}link_paraproximal_bar"/>
@@ -442,7 +442,7 @@
     <gazebo reference="${prefix}joint_paraproximal_bar">
       <implicitSpringDamper>1</implicitSpringDamper>
-    </gazebo>
+    </gazebo> -->
     <!-- Joint median actuating hinge -->
-    <joint name="${prefix}joint_median_actuating_hinge" type="revolute">
+    <!-- <joint name="${prefix}joint_median_actuating_hinge" type="revolute">
       <parent link="${prefix}link_1"/>
       <child link="${prefix}link_median_actuating_hinge"/>
@@ -453,11 +453,11 @@
     <gazebo reference="${prefix}joint_median_actuating_hinge">
       <implicitSpringDamper>1</implicitSpringDamper>
-    </gazebo>
+    </gazebo> -->
     <!-- Joint paramedian hinge -->
-    <joint name="${prefix}joint_paramedian_hinge" type="revolute">
+    <!-- <joint name="${prefix}joint_paramedian_hinge" type="revolute">
       <parent link="${prefix}link_1"/>
       <child link="${prefix}link_paramedian_hinge"/>
       <axis xyz="0 0 1"/>
-      <!-- -0.37 is hand picked, 0.9719 is hand calculated from atan(0.02381/0.01625) -->
+      -0.37 is hand picked, 0.9719 is hand calculated from atan(0.02381/0.01625)
       <origin rpy="0 0 0" xyz="0 0.05715 -0.01"/>
       <limit effort="100" lower="-3.1416" upper="3.1416" velocity="100"/>
@@ -465,11 +465,11 @@
     <gazebo reference="${prefix}joint_paramedian_hinge">
       <implicitSpringDamper>1</implicitSpringDamper>
-    </gazebo>
+    </gazebo> -->
     <!-- Joint median actuating hinge median bar -->
-    <joint name="${prefix}joint_median_actuating_hinge_median_bar" type="revolute">
+    <!-- <joint name="${prefix}joint_median_actuating_hinge_median_bar" type="revolute">
       <parent link="${prefix}link_median_actuating_hinge"/>
       <child link="${prefix}link_median_bar"/>
       <axis xyz="0 0 1"/>
-      <!-- hand calc 90 deg + atan(0.01516/0.01625) -->
+      hand calc 90 deg + atan(0.01516/0.01625)
       <origin rpy="0 0 ${3.1416/2 + 0.7507}" xyz="0.01625 0.01516 0"/>
       <limit effort="100" lower="-3.1416" upper="3.1416" velocity="100"/>
@@ -477,7 +477,7 @@
     <gazebo reference="${prefix}joint_median_actuating_hinge_median_bar">
       <implicitSpringDamper>1</implicitSpringDamper>
-    </gazebo>
+    </gazebo> -->
     <!-- Joint paradistal hinge -->
-    <joint name="${prefix}joint_paradistal_hinge" type="revolute">
+    <!-- <joint name="${prefix}joint_paradistal_hinge" type="revolute">
       <parent link="${prefix}link_2"/>
       <child link="${prefix}link_paradistal_hinge"/>
@@ -488,11 +488,11 @@
     <gazebo reference="${prefix}joint_paradistal_hinge">
       <implicitSpringDamper>1</implicitSpringDamper>
-    </gazebo>
+    </gazebo> -->
     <!-- Joint paramedian hinge median bar underactuated -->
-    <joint name="${prefix}joint_paramedian_hinge_median_bar_underactuated" type="revolute">
+    <!-- <joint name="${prefix}joint_paramedian_hinge_median_bar_underactuated" type="revolute">
       <parent link="${prefix}link_paramedian_hinge"/>
       <child link="${prefix}link_median_bar_underactuated"/>
       <axis xyz="0 0 1"/>
-      <!-- hand calc 90 deg + atan(0.01227/0.00329) -->
+      hand calc 90 deg + atan(0.01227/0.00329)
       <origin rpy="0 0 ${3.1416/2}" xyz="0.01227 0.00329 0"/>
       <limit effort="100" lower="-3.1416" upper="3.1416" velocity="100"/>
@@ -500,5 +500,5 @@
     <gazebo reference="${prefix}joint_paramedian_hinge_median_bar_underactuated">
       <implicitSpringDamper>1</implicitSpringDamper>
-    </gazebo>
+    </gazebo> -->
     <!-- Joint 1 -->
     <joint name="${prefix}joint_1" type="revolute">
@@ -509,9 +509,9 @@
       <dynamics damping="1" friction="0" />
       <!-- Limits: [0deg.,70deg.] -->
-      <limit effort="60" velocity="-1" lower="0" upper="1.2217" />
-    </joint>
-    <gazebo reference="${prefix}joint_1">
-      <implicitSpringDamper>1</implicitSpringDamper>
-    </gazebo>
+      <limit effort="60" velocity="100" lower="0" upper="1.2217" />
+    </joint>
+    <!-- <gazebo reference="${prefix}joint_1">
+      <implicitSpringDamper>1</implicitSpringDamper>
+    </gazebo> -->
     <!-- Joint 2 -->
     <joint name="${prefix}joint_2" type="revolute">
@@ -522,10 +522,10 @@
       <origin rpy="0 0 0" xyz="0 0.05715 0"/>
       <!-- Limits: [0deg.,90deg.] -->
-      <limit lower="0" upper="1.5708" effort="60" velocity="-1"/>
+      <limit lower="0" upper="1.5708" effort="60" velocity="100"/>
       <mimic joint="${prefix}joint_1" multiplier="1" offset="0" />
     </joint>
-    <gazebo reference="${prefix}joint_2">
-      <implicitSpringDamper>1</implicitSpringDamper>
-    </gazebo>
+    <!-- <gazebo reference="${prefix}joint_2">
+      <implicitSpringDamper>1</implicitSpringDamper>
+    </gazebo> -->
     <!-- Joint 3 -->
     <joint name="${prefix}joint_3" type="revolute">
@@ -536,13 +536,13 @@
       <origin rpy="0 0 ${3.1416/2 + 0.5198}" xyz="0 0.039 0"/>
       <!-- Limits: [-38deg.,60deg.] -->
-      <limit lower="-0.6632" upper="1.0471" effort="60" velocity="-1"/>
+      <limit lower="-0.6632" upper="1.0471" effort="60" velocity="100"/>
       <mimic joint="${prefix}joint_2" multiplier="-2" offset="0" />
     </joint>
-    <gazebo reference="${prefix}joint_3">
-      <implicitSpringDamper>1</implicitSpringDamper>
-    </gazebo>
+    <!-- <gazebo reference="${prefix}joint_3">
+      <implicitSpringDamper>1</implicitSpringDamper>
+    </gazebo> -->
     <!-- end of joint list -->
     <!-- coupling joints in sdf -->
-    <gazebo>
+    <!-- <gazebo>
       <joint name="${prefix}link_proximal_actuating_bar_median_actuating_hinge_couple" type="revolute">
         <parent>${prefix}link_median_actuating_hinge</parent>
@@ -555,5 +555,5 @@
           </dynamics>
           <xyz>0 0 1</xyz>
-          <!-- <use_parent_model_frame>false</use_parent_model_frame> -->
+          <use_parent_model_frame>false</use_parent_model_frame>
         </axis>
       </joint>
@@ -561,6 +561,6 @@
     <gazebo reference="${prefix}link_proximal_actuating_bar_median_actuating_hinge_couple">
       <implicitSpringDamper>1</implicitSpringDamper>
-    </gazebo>
-    <gazebo>
+    </gazebo> -->
+    <!-- <gazebo>
       <joint name="${prefix}link_median_bar_link_3_couple" type="revolute">
         <parent>${prefix}link_3</parent>
@@ -573,5 +573,5 @@
           </dynamics>
           <xyz>0 0 1</xyz>
-          <!-- <use_parent_model_frame>false</use_parent_model_frame> -->
+          <use_parent_model_frame>false</use_parent_model_frame>
         </axis>
       </joint>
@@ -579,6 +579,6 @@
     <gazebo reference="${prefix}link_median_bar_link_3_couple">
       <implicitSpringDamper>1</implicitSpringDamper>
-    </gazebo>
-    <gazebo>
+    </gazebo> -->
+    <!-- <gazebo>
       <joint name="${prefix}link_paramedian_bar_paradistal_hinge_couple" type="revolute">
         <parent>${prefix}link_paradistal_hinge</parent>
@@ -591,5 +591,5 @@
           </dynamics>
           <xyz>0 0 1</xyz>
-           <!-- <use_parent_model_frame>false</use_parent_model_frame> -->
+           <use_parent_model_frame>false</use_parent_model_frame>
         </axis>
       </joint>
@@ -597,6 +597,6 @@
     <gazebo reference="${prefix}link_median_bar_link_3_couple">
       <implicitSpringDamper>1</implicitSpringDamper>
-    </gazebo>
-    <gazebo>
+    </gazebo> -->
+    <!-- <gazebo>
       <joint name="${prefix}link_paradistal_hinge_link_3_couple" type="revolute">
         <parent>${prefix}link_paradistal_hinge</parent>
@@ -609,5 +609,5 @@
           </dynamics>
           <xyz>0 0 1</xyz>
-          <!-- <use_parent_model_frame>false</use_parent_model_frame> -->
+          <use_parent_model_frame>false</use_parent_model_frame>
         </axis>
       </joint>
@@ -615,8 +615,10 @@
     <gazebo reference="${prefix}link_paradistal_hinge_link_3_couple">
       <implicitSpringDamper>1</implicitSpringDamper>
+    </gazebo> -->
+    <!-- <gazebo>
+      <joint name="${prefix}link_paraproximal_bar_paramedian_hinge_couple" type="revolute">
+        <parent>${prefix}link_paramedian_hinge</parent>    <gazebo reference="${prefix}joint_1">
+      <implicitSpringDamper>1</implicitSpringDamper>
     </gazebo>
-    <gazebo>
-      <joint name="${prefix}link_paraproximal_bar_paramedian_hinge_couple" type="revolute">
-        <parent>${prefix}link_paramedian_hinge</parent>
         <child>${prefix}link_paraproximal_bar</child>
         <pose>0.05770 0 0 0 0 0</pose>
@@ -627,5 +629,5 @@
           </dynamics>
           <xyz>0 0 1</xyz>
-          <!-- <use_parent_model_frame>false</use_parent_model_frame> -->
+          <use_parent_model_frame>false</use_parent_model_frame>
         </axis>
       </joint>
@@ -633,5 +635,5 @@
     <gazebo reference="${prefix}link_paraproximal_bar_paramedian_hinge_couple">
       <implicitSpringDamper>1</implicitSpringDamper>
-    </gazebo>
+    </gazebo> -->
   </xacro:macro>
   <xacro:macro name="robotiq_hand" params="prefix *origin reflect parent">
@@ -673,8 +675,8 @@
         </inertial>
       </link>
-      <gazebo reference="${prefix}palm">
+      <!-- <gazebo reference="${prefix}palm">
         <mu1>1.1</mu1>
         <mu2>1.1</mu2>
-      </gazebo>
+      </gazebo> -->
     <!-- End of link list -->
     <!-- Joint list -->
@@ -687,9 +689,9 @@
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
File: ros_models/urdfs/ur5e_robotiq_3f.urdf.xacro (robot description, xacro)
@@ -11,4 +11,5 @@
   <!-- robotiq -->
   <xacro:include filename="$(find bulldog_mujoco_ros)/ros_models/urdfs/robotiq_3f/robotiq-3f-gripper_articulated_macro.xacro" />
+  <xacro:include filename="$(find bulldog_mujoco_ros)/ros_models/urdfs/robotiq_3f/robotiq_hand_macro.urdf.xacro" />
   <!-- <body name="robot0_base" pos="-0.56 0.0 0.913">
       <inertial diaginertia="0 0 0" mass="0" pos="0 0 0" />
@@ -119,18 +120,18 @@
     <origin xyz="0 0.082 0" rpy="-1.5708 0 0" />
   </joint>
-  <!-- <xacro:robotiq_hand prefix="gripper0_" parent="robot0_right_hand" reflect="1">
+  <xacro:robotiq_hand prefix="gripper0_" parent="robot0_right_hand" reflect="1">
     <origin xyz="0 0 0.065" rpy="1.5708 0 2.3562" />
-  </xacro:robotiq_hand> -->
-  <xacro:robotiq-3f-gripper_articulated prefix="gripper0_"/>
+  </xacro:robotiq_hand>
+  <!-- <xacro:robotiq-3f-gripper_articulated prefix="gripper0_"/>
   <joint name="gripper0_palm_joint" type="fixed">
     <parent link="robot0_right_hand" />
     <child link="gripper0_palm" />
     <origin xyz="0 0 0.065" rpy="1.5708 0 2.3562" />
-  </joint>
-  <!-- <link name="gripper0_tool0" />
+  </joint> -->
+  <link name="gripper0_tool0" />
   <joint name="gripper0_tool0_joint" type="fixed">
     <parent link="gripper0_palm" />
     <child link="gripper0_tool0" />
     <origin xyz="0 0.1 0" rpy="0 0 0" />
-  </joint> -->
+  </joint>
 </robot>
