Commit message: add panda xml and urdf

File: ros_models/urdfs/panda/panda.transmission.xacro (robot description, xacro)
@@ -1,5 +1,5 @@
 <?xml version="1.0"?>
 <robot xmlns:xacro="http://www.ros.org/wiki/xacro">
-    <xacro:macro name="panda_transmission" params="robot_name load_gripper use_gazebo_control">
+    <xacro:macro name="panda_transmission" params="robot_name gripper_name load_gripper use_gazebo_control">
         <!-- Load Gazebo lib and set the robot namespace -->
         <xacro:if value="${use_gazebo_control}">
@@ -22,4 +22,5 @@
             </gazebo>
         </xacro:unless>
+        <!-- Hardware Interface inside actuator prevents mujoco_ros_control to load transmission -->
         <transmission name="${robot_name}_tran_1">
             <type>transmission_interface/SimpleTransmission</type>
@@ -28,5 +29,5 @@
             </joint>
             <actuator name="${robot_name}_motor_1">
-                <hardwareInterface>hardware_interface/EffortJointInterface</hardwareInterface>
+                <!-- <hardwareInterface>hardware_interface/EffortJointInterface</hardwareInterface> -->
                 <mechanicalReduction>1</mechanicalReduction>
             </actuator>
@@ -38,5 +39,5 @@
             </joint>
             <actuator name="${robot_name}_motor_2">
-                <hardwareInterface>hardware_interface/EffortJointInterface</hardwareInterface>
+                <!-- <hardwareInterface>hardware_interface/EffortJointInterface</hardwareInterface> -->
                 <mechanicalReduction>1</mechanicalReduction>
             </actuator>
@@ -48,5 +49,5 @@
             </joint>
             <actuator name="${robot_name}_motor_3">
-                <hardwareInterface>hardware_interface/EffortJointInterface</hardwareInterface>
+                <!-- <hardwareInterface>hardware_interface/EffortJointInterface</hardwareInterface> -->
                 <mechanicalReduction>1</mechanicalReduction>
             </actuator>
@@ -58,5 +59,5 @@
             </joint>
             <actuator name="${robot_name}_motor_4">
-                <hardwareInterface>hardware_interface/EffortJointInterface</hardwareInterface>
+                <!-- <hardwareInterface>hardware_interface/EffortJointInterface</hardwareInterface> -->
                 <mechanicalReduction>1</mechanicalReduction>
             </actuator>
@@ -68,5 +69,5 @@
             </joint>
             <actuator name="${robot_name}_motor_5">
-                <hardwareInterface>hardware_interface/EffortJointInterface</hardwareInterface>
+                <!-- <hardwareInterface>hardware_interface/EffortJointInterface</hardwareInterface> -->
                 <mechanicalReduction>1</mechanicalReduction>
             </actuator>
@@ -78,5 +79,5 @@
             </joint>
             <actuator name="${robot_name}_motor_6">
-                <hardwareInterface>hardware_interface/EffortJointInterface</hardwareInterface>
+                <!-- <hardwareInterface>hardware_interface/EffortJointInterface</hardwareInterface> -->
                 <mechanicalReduction>1</mechanicalReduction>
             </actuator>
@@ -88,26 +89,26 @@
             </joint>
             <actuator name="${robot_name}_motor_7">
-                <hardwareInterface>hardware_interface/EffortJointInterface</hardwareInterface>
+                <!-- <hardwareInterface>hardware_interface/EffortJointInterface</hardwareInterface> -->
                 <mechanicalReduction>1</mechanicalReduction>
             </actuator>
         </transmission>
         <xacro:if value="${load_gripper}">
-            <transmission name="${robot_name}_leftfinger">
+            <transmission name="${gripper_name}_leftfinger">
                 <type>transmission_interface/SimpleTransmission</type>
-                <joint name="${robot_name}_finger_joint1">
+                <joint name="${gripper_name}_finger_joint1">
                     <hardwareInterface>hardware_interface/EffortJointInterface</hardwareInterface>
                 </joint>
-                <actuator name="${robot_name}_finger_joint1">
-                    <hardwareInterface>hardware_interface/EffortJointInterface</hardwareInterface>
+                <actuator name="${gripper_name}_finger_joint1">
+                    <!-- <hardwareInterface>hardware_interface/EffortJointInterface</hardwareInterface> -->
                     <mechanicalReduction>1</mechanicalReduction>
                 </actuator>
             </transmission>
-            <transmission name="${robot_name}_rightfinger">
+            <transmission name="${gripper_name}_rightfinger">
                 <type>transmission_interface/SimpleTransmission</type>
-                <joint name="${robot_name}_finger_joint2">
+                <joint name="${gripper_name}_finger_joint2">
                     <hardwareInterface>hardware_interface/EffortJointInterface</hardwareInterface>
                 </joint>
-                <actuator name="${robot_name}_finger_joint2">
-                    <hardwareInterface>hardware_interface/EffortJointInterface</hardwareInterface>
+                <actuator name="${gripper_name}_finger_joint2">
+                    <!-- <hardwareInterface>hardware_interface/EffortJointInterface</hardwareInterface> -->
                     <mechanicalReduction>1</mechanicalReduction>
                 </actuator>
