Commit message: add panda_moveit_planning_and_execution.launch

File: ros_models/urdfs/panda/hand.xacro (robot description, xacro)
@@ -92,5 +92,6 @@
       <axis xyz="0 -1 0"/>
       <limit effort="20" lower="0.0" upper="0.04" velocity="0.2"/>
-      <mimic joint="${ns}_finger_joint1" />
+      <!-- to make MuJOCO work -->
+      <!-- <mimic joint="${ns}_finger_joint1" /> -->
     </joint>
   </xacro:macro>
